File: build/WEASEL_KiCad/WEASEL_KiCad.kicad_pcb (KiCad board)
At the start: 2 copper layers, 342.8 x 184 mm, 129 parts, among them J1 MIDI IN, J10 LPG_LEVEL2CTRL, J14 SEQ_OUTPUT2, J15 SEQ_OUTPUT3, J16 EG_OUTPUT1, J17 EG_OUTPUT2, J18 EG_OUTPUT3, J19 PLSR_OUTPUT1, J2 STEREO_OUTPUT, J20 PLSR_OUTPUT2, J21 PLSR_OUTPUT3, J22 RNDM_OUTPUT1, J23 RNDM_OUTPUT2, J24 RNDM_OUTPUT3, J3 SEQ_OUTPUT1, J4 PLSR_PERIODCTRL, J5 MODOSC_FREQCTRL, J6 MODOSC_MODCTRL, J7 COMPOSC_PITCHCTRL, J8 COMPOSC_WAVEFOLDERCTRL, J9 LPG_LEVEL1CTRL, SW1 SQ_TOGGLESTEP1, SW2 SEQ_TRIGGERSELECT, SW3 SQ_TOGGLESTEP2, SW31 EG_TRIGGERSELECT, SW32 EG_MODESELECT, SW33 PLSR_TRIGGERSELECT, SW34 PLSR_MODE, SW35 MODOSC_MIDITOGGLE, SW36 MODOSC_PITCHTRANGE, SW37 COMPLEXOSC_MIDITOGGLE, SW38 COMPLEXOSC_POLARITY, SW39 COMPLEXOSC_WAVETOGGLE, SW4 SQ_TOGGLESTEP3, SW40 LPG_GATE1MODE, SW41 LPG_GATE2MODE, SW42 RNDMVOLTAGE_TRIGGERSELECT, SW43 CLOCK_SYNCTOGGLE, SW5 SQ_TOGGLESTEP4, SW6 SEQ_STAGES, SW7 SQ_TOGGLESTEP5, U1 CD74HC4067, U2 CD74HC4067, U3 6N138

Commit message: PCB & Schematic update
- Removed unnecessary capacitors for each pot. Each MUX signal pin has a capacitor to filter the signal.
- New board layout
- More compact and organised.
Parts:
- removed C10, C11, C12, C13, C14, C15, C16, C17, C18, C19, C20, C21, C22, C23, C24, C25, C26, C27, C3, C4, C5, C6, C7, C8, C9: 10nF, DIYSynthMNL:C_Rect_L7.0mm_W2.0mm_P5.00mm_BigPads
- added ?: , , F.Cu at (29.0, 32.0)
- added ?: , , F.Cu at (312.8, 193.0)
- added ?: , , F.Cu at (29.0, 193.0)
- added G***: LOGO, AXS_LOGO_KICAD:AXS_LOGO_FMASK_20X20, F.Cu at (153.3, 35.9)
- added REF**: MountingHole_M3_Standoff, DIYSynthMNL:MountingHole_M3_Standoff, F.Cu at (321.5, 23.0)
- C1, C2: footprint DIYSynthMNL:C_Rect_L7.0mm_W2.0mm_P5.00mm_BigPads -> PCM_4ms_Capacitor:C_Disc_P5.08mm
- moved D1 286.9 mm to (64.8, 154.0), turned to 180 degrees
- moved D2 248.6 mm to (107.3, 153.5), turned to 180 degrees
- moved D3 238.4 mm to (119.8, 153.5), turned to 180 degrees
- moved D4 228.5 mm to (132.3, 153.5), turned to 180 degrees
- moved D6 218.9 mm to (144.8, 153.5), turned to 180 degrees
- moved D7 185.1 mm to (187.3, 153.5), turned to 180 degrees
- moved D8 177.1 mm to (199.8, 153.5), turned to 180 degrees
- moved D35 173.2 mm to (39.5, 94.0)
- moved SW35 159.7 mm to (46.0, 99.2)
- moved D36 136.8 mm to (56.0, 93.9)
- moved RV14 135.4 mm to (92.6, 124.2), turned to 90 degrees
- moved RV13 131.8 mm to (76.2, 124.2), turned to 90 degrees
- moved RV12 128.2 mm to (59.9, 124.2), turned to 90 degrees
- moved RV11 124.6 mm to (43.5, 124.2), turned to 90 degrees
- moved SW36 123.4 mm to (62.4, 99.2)
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Connections:
- A1 pad 13: B0 -> X0
- A1 pad 14: B0 -> X1
- A1 pad 24: B0 -> X2
- A1 pad 25: B0 -> X3
- A1 pad 27: B0 -> B1
- A1 pad 28: B0 -> B2
- A1 pad 29: B0 -> B3
- A1 pad 38: B0 -> Vcc
- C1 pad 1: Net-(U1-i0) -> MUX2_SIGNAL
- C2 pad 1: Net-(U1-i1) -> MUX1_SIGNAL
- J16 pad S: B0 -> B1
- J16 pad T: B0 -> B1
- J16 pad TN: B0 -> B1
- J17 pad S: B0 -> B1
- J17 pad T: B0 -> B1
- J17 pad TN: B0 -> B1
- J18 pad S: B0 -> B1
- J18 pad T: B0 -> B1
- J18 pad TN: B0 -> B1
- J19 pad S: B0 -> B2
- J19 pad T: B0 -> B2
- J19 pad TN: B0 -> B2
- J20 pad S: B0 -> B2
- J20 pad T: B0 -> B2
- J20 pad TN: B0 -> B2
- J21 pad S: B0 -> B2
- J21 pad T: B0 -> B2
- J21 pad TN: B0 -> B2
- J22 pad S: B0 -> B3
- J22 pad T: B0 -> B3
- J22 pad TN: B0 -> B3
- J23 pad S: B0 -> B3
- J23 pad T: B0 -> B3
- J23 pad TN: B0 -> B3
- J24 pad S: B0 -> B3
- J24 pad T: B0 -> B3
- J24 pad TN: B0 -> B3
- R9 pad 1: B0 -> Vcc
- RV1 pad 3: B0 -> Vcc
- RV10 pad 3: B0 -> Vcc
- RV11 pad 3: B0 -> Vcc
- RV12 pad 1: B0 -> Vcc
- RV13 pad 3: B0 -> Vcc
- RV14 pad 3: B0 -> Vcc
- RV15 pad 3: B0 -> Vcc
- RV16 pad 3: B0 -> Vcc
- RV17 pad 3: B0 -> Vcc
- RV18 pad 3: B0 -> Vcc
- RV19 pad 3: B0 -> Vcc
- RV2 pad 3: B0 -> Vcc
- RV20 pad 3: B0 -> Vcc
- RV21 pad 3: B0 -> Vcc
- RV22 pad 3: B0 -> Vcc
- RV23 pad 3: B0 -> Vcc
- RV24 pad 3: B0 -> Vcc
- RV25 pad 3: B0 -> Vcc
- RV26 pad 3: B0 -> Vcc
- RV27 pad 3: B0 -> Vcc
- RV3 pad 3: B0 -> Vcc
- RV4 pad 3: B0 -> Vcc
- RV5 pad 3: B0 -> Vcc
- RV6 pad 3: B0 -> Vcc
- RV7 pad 3: B0 -> Vcc
- RV8 pad 3: B0 -> Vcc
- RV9 pad 3: B0 -> Vcc
- SW1 pad 2: B0 -> X3
- SW2 pad 1: B0 -> X0
- SW3 pad 2: B0 -> X0
- SW31 pad 1: B0 -> X2
- SW32 pad 1: B0 -> X3
- SW33 pad 1: B0 -> X0
- SW34 pad 1: B0 -> X1
- SW35 pad 1: B0 -> X2
- SW36 pad 1: B0 -> X3
- SW37 pad 1: B0 -> X0
- SW38 pad 1: B0 -> X1
- SW39 pad 1: B0 -> X2
- SW4 pad 2: B0 -> X1
- SW40 pad 1: B0 -> X3
- SW41 pad 1: B0 -> X0
- SW42 pad 1: B0 -> X1
- SW43 pad 1: B0 -> X2
- SW5 pad 2: B0 -> X2
- SW6 pad 1: B0 -> X1
- SW7 pad 2: B0 -> X3
- U1 pad EN: (no net) -> GND
- U1 pad GND: (no net) -> GND
- U2 pad EN: (no net) -> GND
- U2 pad GND: (no net) -> GND
- U3 pad 8: B0 -> Vcc
Routing:
- net B0: track 3942.3 -> 529.5 mm, vias 22 -> 0
- net (no net): track 1390.5 -> 0.00 mm
- net Vcc: track 0.00 -> 1071.8 mm, vias 0 -> 6
- net Net-(D8-A): track 688.7 -> 16.5 mm, vias 1 -> 0
- net Net-(D7-A): track 671.3 -> 16.5 mm, vias 1 -> 0
- net B2: track 0.00 -> 584.4 mm
- net B3: track 0.00 -> 556.4 mm
- net B1: track 0.00 -> 522.1 mm
- net X2: track 0.00 -> 465.7 mm, vias 0 -> 5
- net X0: track 0.00 -> 446.5 mm, vias 0 -> 10
- net X3: track 0.00 -> 444.0 mm, vias 0 -> 9
- net A0: track 3.45 -> 421.1 mm
- net MUX1_S1: track 712.3 -> 309.3 mm, vias 1 -> 2
- net MUX1_S0: track 707.1 -> 316.2 mm, vias 1 -> 2
- net X1: track 0.00 -> 388.1 mm, vias 0 -> 5
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Other:
- board size 342.8 x 184 mm -> 309.8 x 179 mm
- board text added: "Digital West Coast Synth Inspired by the MUSIC EASEL"
- board text added: "Main Board"
- board text added: "WEASEL"
- board text removed: "LINE OUT"
- board text removed: "MIDI IN"

Commit message: Front panel PCB
Parts:
- added REF**: PanelHole_AudioJack_3.5mm, DIYSynthMNL:PanelHole_AudioJack_3.5mm, F.Cu at (156.0, 343.7)
- added REF**: PanelHole_Potentiometer_RV09, DIYSynthMNL:PanelHole_Potentiometer_RV09, F.Cu at (59.9, 266.2)
- added REF**: PanelHole_Potentiometer_RV09, DIYSynthMNL:PanelHole_Potentiometer_RV09, F.Cu at (76.2, 303.2)
- added REF**: pushbuttonSwitch_6mm, DIYSynthMNL:PanelHole_ToggleSwitch_MTS-101, F.Cu at (179.2, 278.2)
- added REF**: PanelHole_Potentiometer_RV09, DIYSynthMNL:PanelHole_Potentiometer_RV09, F.Cu at (92.6, 303.2)
- added REF**: PanelHole_Potentiometer_RV09, DIYSynthMNL:PanelHole_Potentiometer_RV09, F.Cu at (145.4, 303.2)
- added REF**: PanelHole_Potentiometer_RV09, DIYSynthMNL:PanelHole_Potentiometer_RV09, F.Cu at (145.2, 266.2)
- added REF**: pushbuttonSwitch_6mm, DIYSynthMNL:PanelHole_ToggleSwitch_MTS-101, F.Cu at (147.7, 243.7)
- added REF**: PanelHole_AudioJack_3.5mm, DIYSynthMNL:PanelHole_AudioJack_3.5mm, F.Cu at (211.0, 329.2)
- added REF**: pushbuttonSwitch_6mm, DIYSynthMNL:PanelHole_ToggleSwitch_MTS-101, F.Cu at (217.1, 278.2)
- added REF**: PanelHole_Potentiometer_RV09, DIYSynthMNL:PanelHole_Potentiometer_RV09, F.Cu at (129.0, 285.7)
- added REF**: PanelHole_Potentiometer_RV09, DIYSynthMNL:PanelHole_Potentiometer_RV09, F.Cu at (161.7, 303.2)
- added REF**: PanelHole_ToggleSwitch_MTS-101, DIYSynthMNL:PanelHole_ToggleSwitch_MTS-101, F.Cu at (78.7, 64.7)
- added REF**: PanelHole_ToggleSwitch_MTS-101, DIYSynthMNL:PanelHole_ToggleSwitch_MTS-101, F.Cu at (111.5, 64.7)
- added REF**: PanelHole_AudioJack_3.5mm, DIYSynthMNL:PanelHole_AudioJack_3.5mm, F.Cu at (103.5, 335.7)
- added REF**: PanelHole_AudioJack_3.5mm, DIYSynthMNL:PanelHole_AudioJack_3.5mm, F.Cu at (183.5, 335.7)
- added REF**: PanelHole_Potentiometer_RV09, DIYSynthMNL:PanelHole_Potentiometer_RV09, F.Cu at (224.6, 246.2)
- added REF**: PanelHole_AudioJack_3.5mm, DIYSynthMNL:PanelHole_AudioJack_3.5mm, F.Cu at (211.0, 343.7)
- added REF**: PanelHole_Potentiometer_RV09, DIYSynthMNL:PanelHole_Potentiometer_RV09, F.Cu at (43.5, 303.2)
- added REF**: PanelHole_Potentiometer_RV09, DIYSynthMNL:PanelHole_Potentiometer_RV09, F.Cu at (76.2, 266.2)
- added REF**: PanelHole_AudioJack_3.5mm, DIYSynthMNL:PanelHole_AudioJack_3.5mm, F.Cu at (76.0, 329.2)
- added REF**: PanelHole_Potentiometer_RV09, DIYSynthMNL:PanelHole_Potentiometer_RV09, F.Cu at (129.0, 266.2)
- added REF**: PanelHole_Potentiometer_RV09, DIYSynthMNL:PanelHole_Potentiometer_RV09, F.Cu at (43.5, 266.2)
- added REF**: pushbuttonSwitch_6mm, DIYSynthMNL:PanelHole_ToggleSwitch_MTS-101, F.Cu at (62.4, 228.7)
- added REF**: PanelHole_AudioJack_3.5mm, DIYSynthMNL:PanelHole_AudioJack_3.5mm, F.Cu at (156.0, 329.2)
- added REF**: PanelHole_Potentiometer_RV09, DIYSynthMNL:PanelHole_Potentiometer_RV09, F.Cu at (112.6, 303.2)
- added REF**: PanelHole_AudioJack_3.5mm, DIYSynthMNL:PanelHole_AudioJack_3.5mm, F.Cu at (46.0, 329.2)
- added REF**: pushbuttonSwitch_6mm, DIYSynthMNL:PanelHole_ToggleSwitch_MTS-101, F.Cu at (180.7, 243.7)
- added REF**: PanelHole_ToggleSwitch_MTS-101, DIYSynthMNL:PanelHole_ToggleSwitch_MTS-101, F.Cu at (62.4, 64.7)
- added REF**: PanelHole_AudioJack_3.5mm, DIYSynthMNL:PanelHole_AudioJack_3.5mm, F.Cu at (168.5, 343.7)
- added REF**: PanelHole_Potentiometer_RV09, DIYSynthMNL:PanelHole_Potentiometer_RV09, F.Cu at (145.4, 285.7)
- added REF**: PanelHole_Potentiometer_RV09, DIYSynthMNL:PanelHole_Potentiometer_RV09, F.Cu at (161.7, 266.2)
- added REF**: pushbuttonSwitch_6mm, DIYSynthMNL:PanelHole_ToggleSwitch_MTS-101, F.Cu at (62.4, 278.2)
- added REF**: PanelHole_Potentiometer_RV09, DIYSynthMNL:PanelHole_Potentiometer_RV09, F.Cu at (181.7, 266.2)
- added REF**: PanelHole_AudioJack_3.5mm, DIYSynthMNL:PanelHole_AudioJack_3.5mm, F.Cu at (168.5, 329.2)
- added REF**: pushbuttonSwitch_6mm, DIYSynthMNL:PanelHole_ToggleSwitch_MTS-101, F.Cu at (46.0, 278.2)
- added REF**: PanelHole_AudioJack_3.5mm, DIYSynthMNL:PanelHole_AudioJack_3.5mm, F.Cu at (128.5, 335.7)
- added REF**: PanelHole_Potentiometer_RV09, DIYSynthMNL:PanelHole_Potentiometer_RV09, F.Cu at (247.4, 303.2)
- added REF**: PanelHole_ToggleSwitch_MTS-101, DIYSynthMNL:PanelHole_ToggleSwitch_MTS-101, F.Cu at (95.1, 64.7)
- added REF**: pushbuttonSwitch_6mm, DIYSynthMNL:PanelHole_ToggleSwitch_MTS-101, F.Cu at (212.1, 238.7)
- added REF**: PanelHole_AudioJack_3.5mm, DIYSynthMNL:PanelHole_AudioJack_3.5mm, F.Cu at (46.0, 343.7)
- added REF**: pushbuttonSwitch_6mm, DIYSynthMNL:PanelHole_ToggleSwitch_MTS-101, F.Cu at (233.5, 278.2)
- added REF**: PanelHole_AudioJack_3.5mm, DIYSynthMNL:PanelHole_AudioJack_3.5mm, F.Cu at (76.0, 343.7)
- added REF**: PanelHole_Potentiometer_RV09, DIYSynthMNL:PanelHole_Potentiometer_RV09, F.Cu at (247.4, 246.2)
- added REF**: PanelHole_AudioJack_3.5mm, DIYSynthMNL:PanelHole_AudioJack_3.5mm, F.Cu at (196.0, 335.7)
- added REF**: PanelHole_Potentiometer_RV09, DIYSynthMNL:PanelHole_Potentiometer_RV09, F.Cu at (129.0, 303.2)
- added REF**: PanelHole_AudioJack_3.5mm, DIYSynthMNL:PanelHole_AudioJack_3.5mm, F.Cu at (61.0, 335.9)
- added REF**: PanelHole_Potentiometer_RV09, DIYSynthMNL:PanelHole_Potentiometer_RV09, F.Cu at (231.0, 303.2)
- added REF**: PanelHole_AudioJack_3.5mm, DIYSynthMNL:PanelHole_AudioJack_3.5mm, F.Cu at (88.5, 329.2)
- added REF**: PanelHole_Potentiometer_RV09, DIYSynthMNL:PanelHole_Potentiometer_RV09, F.Cu at (198.2, 303.2)
- added REF**: pushbuttonSwitch_6mm, DIYSynthMNL:PanelHole_ToggleSwitch_MTS-101, F.Cu at (164.2, 278.2)
- added REF**: pushbuttonSwitch_6mm, DIYSynthMNL:PanelHole_ToggleSwitch_MTS-101, F.Cu at (46.0, 228.7)
- added REF**: PanelHole_Potentiometer_RV09, DIYSynthMNL:PanelHole_Potentiometer_RV09, F.Cu at (214.6, 303.2)
- added REF**: PanelHole_Potentiometer_RV09, DIYSynthMNL:PanelHole_Potentiometer_RV09, F.Cu at (109.0, 266.2)
- added REF**: PanelHole_Potentiometer_RV09, DIYSynthMNL:PanelHole_Potentiometer_RV09, F.Cu at (198.2, 266.2)
- added REF**: PanelHole_Potentiometer_RV09, DIYSynthMNL:PanelHole_Potentiometer_RV09, F.Cu at (92.6, 285.7)
- added REF**: PanelHole_Potentiometer_RV09, DIYSynthMNL:PanelHole_Potentiometer_RV09, F.Cu at (59.9, 303.2)
- added REF**: PanelHole_AudioJack_3.5mm, DIYSynthMNL:PanelHole_AudioJack_3.5mm, F.Cu at (116.0, 335.7)
- added REF**: PanelHole_Potentiometer_RV09, DIYSynthMNL:PanelHole_Potentiometer_RV09, F.Cu at (92.6, 266.2)
- added REF**: pushbuttonSwitch_6mm, DIYSynthMNL:PanelHole_ToggleSwitch_MTS-101, F.Cu at (131.5, 243.7)
- added REF**: pushbuttonSwitch_6mm, DIYSynthMNL:PanelHole_ToggleSwitch_MTS-101, F.Cu at (164.2, 243.7)
- added REF**: PanelHole_AudioJack_3.5mm, DIYSynthMNL:PanelHole_AudioJack_3.5mm, F.Cu at (141.0, 335.7)
- added REF**: PanelHole_AudioJack_3.5mm, DIYSynthMNL:PanelHole_AudioJack_3.5mm, F.Cu at (88.5, 343.7)
- added REF**: PanelHole_ToggleSwitch_MTS-101, DIYSynthMNL:PanelHole_ToggleSwitch_MTS-101, F.Cu at (46.0, 64.7)
- added REF**: pushbuttonSwitch_6mm, DIYSynthMNL:PanelHole_ToggleSwitch_MTS-101, F.Cu at (233.5, 258.7)
Other:
- board size 309.8 x 179 mm -> 309.8 x 537 mm
