File: build/WEASEL_KiCad/WEASEL_KiCad.kicad_sch (KiCad schematic)
At the start: 104 parts, among them J1 MIDI IN, J10 PLSR_OUTPUT2, J11 PLSR_OUTPUT3, J12 RNDM_OUTPUT1, J13 RNDM_OUTPUT2, J14 RNDM_OUTPUT3, J15 PLSR_PERIODCTRL, J16 MODOSC_FREQCTRL, J17 MODOSC_MODCTRL, J18 COMPOSC_PITCHCTRL, J19 COMPOSC_WAVEFOLDERCTRL, J2 STEREO_OUTPUT, J20 LPG_LEVEL1CTRL, J21 LPG_LEVEL2CTRL, J22 Jack-DC, J3 SEQ_OUTPUT1, J4 SEQ_OUTPUT2, J5 SEQ_OUTPUT3, J6 EG_OUTPUT1, J7 EG_OUTPUT2, J8 EG_OUTPUT3, J9 PLSR_OUTPUT1, SW1 SEQ_TRIGGERSELECT, SW10 COMPLEXOSC_POLARITY, SW11 COMPLEXOSC_WAVETOGGLE, SW12 LPG_GATE1MODE, SW13 LPG_GATE2MODE, SW14 RNDMVOLTAGE_TRIGGERSELECT, SW15 CLOCK_SYNCTOGGLE, SW16 SQ_TOGGLESTEP1, SW17 SQ_TOGGLESTEP2, SW18 SQ_TOGGLESTEP3, SW19 SQ_TOGGLESTEP4, SW2 SEQ_STAGES, SW20 SQ_TOGGLESTEP5, SW3 EG_TRIGGERSELECT, SW4 EG_MODESELECT, SW5 PLSR_TRIGGERSELECT, SW6 PLSR_MODE, SW7 MODOSC_MODULATIONMODE, SW8 MODOSC_WAVEFORMTOGGLE, SW9 OSCILLATOR_MIDITOGGLE, U1 CD74HC4067, U2 CD74HC4067, U3 6N138

Commit message: PCB & Schematic Changes
Added Shift registers for buttons
Added I2C LED Drivers for better visual feedback
- Removed Button matrices
Parts:
- removed D14, D15, D16, D17, D18, D19, D20, D21, D22, D3, D4, D5, D6, D7, D8, D9: 1N4148, DIYSynthMNL:D_4148_BigPads, symbol PCM_4ms_Diode:D_Generic
- removed U1, U2: CD74HC4067, CD74HC4067 MUX:CD74HC4067_matchesSymbol, symbol CD74HC4067:CD74HC4067
- added C1, C2, C31, C34, C35, C36, C37, C38, C39, C40, C41: 100nF_0603_16V, Capacitor_SMD:C_1206_3216Metric, symbol PCM_4ms_Capacitor:100nF_0603_16V
- added C10, C11, C12, C13, C14, C15, C16, C17, C18, C19, C20, C21, C22, C23, C24, C25, C26, C27, C28, C29, C3, C30, C4, C5, C6, C7, C8, C9: C_Generic, Capacitor_SMD:C_1206_3216Metric_Pad1.33x1.80mm_HandSolder, symbol PCM_4ms_Capacitor:C_Generic
- added C32: 10uF, Capacitor_SMD:C_1206_3216Metric_Pad1.33x1.80mm_HandSolder, symbol Device:C
- added C33: 100uF_25V, Capacitor_THT:CP_Radial_D6.3mm_P2.50mm, symbol PCM_SL_Capacitors:100uF_25V
- added D14, D15, D16, D17, D18, D19, D20, D21, D22, D3, D30, D31, D32, D33, D34, D35, D36, D37, D38, D39, D4, D40, D41, D42, D43, D44, D45, D46, D47, D48, D49, D5, D50, D51, D52, D53, D54, D55, D56, D57, D58, D59, D6, D60, D61, D62, D63, D64, D65, D7, D8, D9: LED, PCM_4ms_LED:LED_0603_1608Metric, symbol Device:LED
- added D2: 1N5817, PCM_Diode_SMD_AKL:D_1206_3216Metric_Pad1.42x1.75mm_HandSolder, symbol PCM_Diode_Schottky_AKL:BAT43
- added F1: 1A_15V, Fuse:Fuse_1812_4532Metric, symbol PCM_4ms_Regulator:Polyfuse_3A_15V
- added R10, R11, R12, R13, R14, R15, R16, R17, R18, R19, R20, R21, R22, R23, R24, R25, R26, R27, R4, R5, R6, R7, R8, R9: 10k_0402, PCM_4ms_Resistor:R_0603, symbol PCM_4ms_Resistor:10k_0402
- added RV28: MASTER, benjiaomodular:Potentiometer_RV09, symbol Device:R_Potentiometer
- added U1, U10, U11, U2: AW9523B, Package_DFN_QFN:QFN-24-1EP_4x4mm_P0.5mm_EP2.7x2.7mm, symbol Interface_Expansion:AW9523B
- added U4, U5: CD74HC4067M, Package_SO:SOIC-24W_7.5x15.4mm_P1.27mm, symbol 74xx:CD74HC4067M
- added U6, U7, U8, U9: 74HC165, Package_SO:SOIC-16_3.9x9.9mm_P1.27mm, symbol 74xx:74HC165
- D1, D10, D11, D12, D13, D23, D24, D25, D26, D27, D28, D29: footprint DIYSynthMNL:D_4148_BigPads -> Diode_SMD:D_SOD-123
- J1, J2: footprint trsSocket:Jack_3.5mm_CUI_SJ1-3523N_Horizontal_edited_noEdgeCuts -> PJ307-TRS:Jack_3.5mm_CUI_SJ1-3525N_Horizontal
- R1: footprint PCM_4ms_Resistor:R_Axial_DIN0207_L6.3mm_D2.5mm_P7.62mm_Horizontal -> PCM_4ms_Resistor:R_0603
- R2: value 220R -> 470R; footprint PCM_4ms_Resistor:R_Axial_DIN0207_L6.3mm_D2.5mm_P7.62mm_Horizontal -> PCM_4ms_Resistor:R_0603
- R3: value 4k7 -> 1k; footprint PCM_4ms_Resistor:R_Axial_DIN0207_L6.3mm_D2.5mm_P7.62mm_Horizontal -> PCM_4ms_Resistor:R_0603
- RV15, RV18, RV21, RV26, RV27: footprint DIYSynthMNL:Potentiometer_RV09_BigPads -> benjiaomodular:Potentiometer_RV09
- U3: footprint DIYSynthMNL:DIP-8_W7.62mm_LongPads -> Package_SO:SOP-8_6.62x9.15mm_P2.54mm
Connections:
- net AGND: now also RV1.1, RV10.1, RV11.1, RV12.1, RV13.1, RV14.1, RV15.1, RV16.1, RV17.1, RV18.1, RV19.1, RV2.1, RV20.1, RV21.1, RV22.1, RV23.1, RV24.1, RV25.1, RV26.1, RV27.1, RV3.1, RV4.1, RV5.1, RV6.1, RV7.1, RV8.1, RV9.1, C1.2, C10.2, C11.2, C12.2, C13.2, C14.2, C15.2, C16.2, C17.2, C18.2, C19.2, C2.2, C20.2, C21.2, C22.2, C23.2, C24.2, C25.2, C26.2, C27.2, C28.2, C29.2, C3.2, C30.2, C4.2, C5.2, C6.2, C7.2, C8.2, C9.2, R4.2, R7.2, RV28.1, U4.12 (GND), U5.12 (GND), U5.16 (I15), U5.17 (I14), U5.18 (I13), U5.19 (I12)
- net MUX1_S0: now also U4.10 (S0)
- net MUX1_S1: now also U4.11 (S1)
- net MUX1_S2: now also U4.14 (S2)
- net MUX1_S3: now also U4.13 (S3)
- net MUX1_SIGNAL: now also U4.1 (COM)
- net MUX2_S0: now also U5.10 (S0)
- net MUX2_S1: now also U5.11 (S1)
- net MUX2_S2: now also U5.14 (S2)
- net MUX2_S3: now also A1.11 (SPI1_PICO), U5.13 (S3); no longer A1.8 (SPI1_CS)
- net MUX2_SIGNAL: now also U5.1 (COM)
- net Vin: now also C31.2, C32.1, C33.1, D2.1 (K); no longer J22.2
- net D3V3: now reaches SW10.2
- net D3V3: now also A1.38 (3V3_D), R2.1, SW1.2, SW11.2, SW12.2, SW13.2, SW14.2, SW15.2, SW16.1 (A), SW17.1 (A), SW18.1 (A), SW19.1 (A), SW2.2, SW20.1 (A), SW3.2, SW4.2, SW5.2, SW6.2, SW7.2, SW8.2, SW9.2, U3.8 (VCC), C34.2, C35.2, C36.1, C37.1, C38.1, C39.1, C40.2, C41.2, R26.1, R27.1, U1.21 (VCC), U10.21 (VCC), U10.24 (AD1), U11.18 (AD0), U11.21 (VCC), U11.24 (AD1), U2.18 (AD0), U2.21 (VCC), U6.16 (VCC), U7.16 (VCC), U8.16 (VCC), U9.16 (VCC); no longer D12.2 (A)
- net RNDM_OUTPUT_PATCH: now reaches D13.2 (A)
- net RNDM_OUTPUT_PATCH: now also A1.27 (ADC_5); no longer SW11.2
- net PLSRCTRL: now reaches RV9.2
- net PLSRCTRL: now also C11.1, U4.23 (I8)
- net MODFINE: now reaches RV15.2
- net MODFINE: now also C15.1, U4.19 (I12)
- net STSTEP3: now reaches RV3.2
- net STSTEP3: now also C5.1, U4.7 (I2)
- net COMPLEXFREQCTRL: now reaches RV16.2
- net COMPLEXFREQCTRL: now also C18.1, U4.16 (I15)
- net MODMOD: now reaches RV14.2
- net MODMOD: now also C17.1, U4.17 (I14)
- net MODMODCTRL: now reaches RV13.2
- net MODMODCTRL: now also C16.1, U4.18 (I13)
- net EGDECAY: now reaches RV8.2
- net EGDECAY: now also C10.1, U4.2 (I7)
- net MODFREQ: now reaches RV12.2
- net MODFREQ: now also C14.1, U4.20 (I11)
- net MODFREQCTRL: now reaches RV11.2
- net MODFREQCTRL: now also C13.1, U4.21 (I10)
- net PLSRPERIOD: now reaches RV10.2
- net PLSRPERIOD: now also C12.1, U4.22 (I9)
- net EGSUS: now reaches RV7.2
- net EGSUS: now also C9.1, U4.3 (I6)
- net EGATT: now reaches RV6.2
- net EGATT: now also C8.1, U4.4 (I5)
- net STSTEP5: now reaches RV5.2
- net STSTEP5: now also C7.1, U4.5 (I4)
- net STSTEP4: now reaches RV4.2
- net STSTEP4: now also C6.1, U4.6 (I3)
- net STSTEP2: now reaches RV2.2
- net STSTEP2: now also C4.1, U4.8 (I1)
- net STSTEP1: now reaches RV1.2
- net STSTEP1: now also C3.1, U4.9 (I0)
- net LPG2CTRL: now reaches RV24.2
- net LPG2CTRL: now also C26.1, U5.2 (I7)
- net LGP1LEVEL: now reaches RV23.2
- net LGP1LEVEL: now also C25.1, U5.3 (I6)
- net REVERB MIX: now reaches RV27.2
- net REVERB MIX: now also C29.1, U5.21 (I10)
- net LGP2LEVEL: now reaches RV25.2
- net LGP2LEVEL: now also C27.1, U5.23 (I8)
- net PLSR_OUTPUT_PATCH: now reaches D11.2 (A)
- net PLSR_OUTPUT_PATCH: now also A1.26 (ADC_4); no longer SW9.2
- net at D24.2 (A), J16.T, J16.TN: no longer J16.S
- net at D26.2 (A), J18.T, J18.TN: no longer J18.S
- net at D27.2 (A), J19.T, J19.TN: no longer J19.S
- net at D29.2 (A), J21.T, J21.TN: no longer J21.S
- net SEQ_OUTPUT_PATCH: now reaches D10.2 (A)
- net SEQ_OUTPUT_PATCH: now also A1.24 (ADC_2); no longer SW8.2
- net at D28.2 (A), J20.T, J20.TN: no longer J20.S
- net COMPLEXWAVE: now reaches RV20.2
- net COMPLEXWAVE: now also C22.1, U5.6 (I3)
- net at D25.2 (A), J17.T, J17.TN: no longer J17.S
- net at D23.2 (A), J15.T, J15.TN: no longer J15.S
- net COMPLEXWAVECTRL: now reaches RV19.2
- net COMPLEXWAVECTRL: now also C21.1, U5.7 (I2)
- net A3V3: now reaches A1.21 (3V3_A)
- net A3V3: now also RV1.3, RV10.3, RV11.3, RV12.3, RV13.3, RV14.3, RV15.3, RV16.3, RV17.3, RV18.3, RV19.3, RV2.3, RV20.3, RV21.3, RV22.3, RV23.3, RV24.3, RV25.3, RV26.3, RV27.3, RV3.3, RV4.3, RV5.3, RV6.3, RV7.3, RV8.3, RV9.3, C1.1, C2.1, RV28.3, U4.24 (VCC), U5.24 (VCC)
- net CLOCK: now reaches RV26.2
- net CLOCK: now also C28.1, U5.22 (I9)
- net LPG1CTRL: now reaches RV22.2
- net LPG1CTRL: now also C24.1, U5.4 (I5)
- net COMPLEXTIMBRE: now reaches RV21.2
- net COMPLEXTIMBRE: now also C23.1, U5.5 (I4)
- net COMPLEXFINE: now reaches RV18.2
- net COMPLEXFINE: now also C20.1, U5.8 (I1)
- net COMPLEXFREQ: now reaches RV17.2
- net COMPLEXFREQ: now also C19.1, U5.9 (I0)
- net A0: no longer names the net of A1.30 (DAC_OUT1)
- net A0: no longer D23.1 (K)
- net A1: no longer names the net of A1.31 (SAI2_MCLK)
- net A1: no longer D24.1 (K)
- net A2: no longer names the net of A1.32 (SAI2_SD_B)
- net A2: no longer D25.1 (K)
- net A3: no longer names the net of A1.33 (SAI2_SD_A)
- net A3: no longer D26.1 (K)
- net A4: no longer names the net of A1.34 (SAI2_FS)
- net A4: no longer D27.1 (K)
- net A5: no longer names the net of A1.35 (SAI2_SCK)
- net A5: no longer D28.1 (K)
- net A6: no longer names the net of A1.36 (USB_D_-)
- net A6: no longer D29.1 (K)
- net B0: no longer names the net of J3.T, J3.TN, J4.T, J4.TN, J5.T, J5.TN
- net B0: now also D10.1 (K); no longer A1.26 (ADC_4), J3.S, J4.S, J5.S
- net B1: no longer names the net of J6.T, J6.TN, J7.T, J7.TN, J8.T, J8.TN
- net B1: now also D12.1 (K); no longer A1.27 (ADC_5), J6.S, J7.S, J8.S
- net B2: no longer names the net of J10.T, J10.TN, J11.T, J11.TN, J9.T, J9.TN
- net B2: now also D11.1 (K); no longer A1.28 (ADC_6), J10.S, J11.S, J9.S
- net B3: no longer names the net of J12.T, J12.TN, J13.T, J13.TN, J14.T, J14.TN
- net B3: now also D13.1 (K); no longer A1.29 (DAC_OUT2), J12.S, J13.S, J14.S
- removed net GND: A1.40 (DGND), J1.S, J22.1, R3.2, RV1.1, RV10.1, RV11.1, RV12.1, RV13.1, RV14.1, RV15.1, RV16.1, RV17.1, RV18.1, RV19.1, RV2.1, RV20.1, RV21.1, RV22.1, RV23.1, RV24.1, RV25.1, RV26.1, RV27.1, RV3.1, RV4.1, RV5.1, RV6.1, RV7.1, RV8.1, RV9.1, U3.5 (GND)
- removed net Vcc: A1.38 (3V3_D), R2.1, RV1.3, RV10.3, RV11.3, RV12.3, RV13.3, RV14.3, RV15.3, RV16.3, RV17.3, RV18.3, RV19.3, RV2.3, RV20.3, RV21.3, RV22.3, RV23.3, RV24.3, RV25.3, RV26.3, RV27.3, RV3.3, RV4.3, RV5.3, RV6.3, RV7.3, RV8.3, RV9.3, U3.8 (VCC)
- removed net X0: A1.13 (I2C1_SDA), SW1.1, SW13.1, SW17.2 (B), SW5.1, SW9.1
- removed net X1: A1.14 (USART1_TX), SW10.1, SW14.1, SW18.2 (B), SW2.1, SW6.1
- removed net X2: A1.24 (ADC_2), SW11.1, SW15.1, SW19.2 (B), SW3.1, SW7.1
- removed net X3: A1.25 (ADC_3), SW12.1, SW16.2 (B), SW20.2 (B), SW4.1, SW8.1
- net Y0 renamed SHIFT_CLOCK
- net SHIFT_CLOCK: now also U6.2 (CP), U7.2 (CP), U8.2 (CP), U9.2 (CP)
- net Y1 renamed SERIAL_OUT
- net SERIAL_OUT: now also U9.9 (Q7); no longer D10.1 (K)
- removed net Y2: A1.11 (SPI1_PICO), D11.1 (K), D12.1 (K), D13.1 (K)
- net Y3 renamed SCL
- net SCL: now also R26.2, U1.19 (SCL), U10.19 (SCL), U11.19 (SCL), U2.19 (SCL)
- net Y4: no longer names the net of A1.37 (USB_D_+)
- new net: D45.2 (A), U2.17 (P1_7)
- new net: D35.2 (A), U2.11 (P0_5)
- new net: D38.2 (A), U2.1 (P1_0)
- new net: D34.2 (A), U2.10 (P0_4)
- new net: D36.2 (A), U2.12 (P0_6)
- new net: D37.2 (A), U2.13 (P0_7)
- new net: D42.2 (A), U2.14 (P1_4)
- new net: D43.2 (A), U2.15 (P1_5)
- new net: D44.2 (A), U2.16 (P1_6)
- new net: D39.2 (A), U2.2 (P1_1)
- new net: D40.2 (A), U2.3 (P1_2)
- new net: D41.2 (A), U2.4 (P1_3)
- new net: D30.2 (A), U2.5 (P0_0)
- new net: D31.2 (A), U2.6 (P0_1)
- new net: D32.2 (A), U2.7 (P0_2)
- new net: D33.2 (A), U2.8 (P0_3)
- new net: R7.1, U4.15 (~{E})
- new net: D55.2 (A), U10.2 (P1_1)
- new net: D58.2 (A), U10.14 (P1_4)
- new net: D49.2 (A), U10.8 (P0_3)
- new net: D57.2 (A), U10.4 (P1_3)
- new net: D47.2 (A), U10.6 (P0_1)
- new net: D61.2 (A), U10.17 (P1_7)
- new net: D20.2 (A), U1.15 (P1_5)
- new net: U6.9 (Q7), U7.10 (DS)
- new net: R4.1, U5.15 (~{E})
- new net: D52.2 (A), U10.12 (P0_6)
- new net: D65.2 (A), U11.8 (P0_3)
- new net: D56.2 (A), U10.3 (P1_2)
- new net: D16.2 (A), U1.2 (P1_1)
- new net: D46.2 (A), U10.5 (P0_0)
- new net: D5.2 (A), U1.7 (P0_2)
- new net: D14.2 (A), U1.13 (P0_7)
- new net: D63.2 (A), U11.6 (P0_1)
- new net: D3.2 (A), U1.5 (P0_0)
- new net: D4.2 (A), U1.6 (P0_1)
- new net: D62.2 (A), U11.5 (P0_0)
- new net: D64.2 (A), U11.7 (P0_2)
- new net: D48.2 (A), U10.7 (P0_2)
- new net: D15.2 (A), U1.1 (P1_0)
- new net: D6.2 (A), U1.8 (P0_3)
- new net: D9.2 (A), U1.12 (P0_6)
- new net: F1.1, J22.2
- new net: D60.2 (A), U10.16 (P1_6)
- new net: D54.2 (A), U10.1 (P1_0)
- new net: D8.2 (A), U1.11 (P0_5)
- new net: D7.2 (A), U1.10 (P0_4)
- new net: D59.2 (A), U10.15 (P1_5)
- new net: D50.2 (A), U10.10 (P0_4)
- new net: D18.2 (A), U1.4 (P1_3)
- new net: D53.2 (A), U10.13 (P0_7)
- new net: D19.2 (A), U1.14 (P1_4)
- new net: D21.2 (A), U1.16 (P1_6)
- new net: U8.9 (Q7), U9.10 (DS)
- new net: D51.2 (A), U10.11 (P0_5)
- new net: D2.2 (A), F1.2
- new net: U7.9 (Q7), U8.10 (DS)
- new net: D22.2 (A), U1.17 (P1_7)
- new net: D17.2 (A), U1.3 (P1_2)
- new net CLOCK_SYNCTOGGLE: R25.1, SW15.1, U7.14 (D3)
- new net COMPLEXOSC_POLARITY: R19.1, SW10.1, U8.4 (D5)
- new net COMPLEXOSC_WAVETOGGLE: R20.1, SW11.1, U8.5 (D6)
- new net COMPOSC_PITCHCTRL: D26.1 (K), U6.14 (D3)
- new net COMPOSC_WAVEFOLDERCTRL: D27.1 (K), U6.3 (D4)
- new net DGND: A1.40 (DGND), C31.1, C32.2, C33.2, C34.1, C35.1, C36.2, C37.2, C38.2, C39.2, C40.1, C41.1, D14.1 (K), D15.1 (K), D16.1 (K), D17.1 (K), D18.1 (K), D19.1 (K), D20.1 (K), D21.1 (K), D22.1 (K), D3.1 (K), D30.1 (K), D31.1 (K), D32.1 (K), D33.1 (K), D34.1 (K), D35.1 (K), D36.1 (K), D37.1 (K), D38.1 (K), D39.1 (K), D4.1 (K), D40.1 (K), D41.1 (K), D42.1 (K), D43.1 (K), D44.1 (K), D45.1 (K), D46.1 (K), D47.1 (K), D48.1 (K), D49.1 (K), D5.1 (K), D50.1 (K), D51.1 (K), D52.1 (K), D53.1 (K), D54.1 (K), D55.1 (K), D56.1 (K), D57.1 (K), D58.1 (K), D59.1 (K), D6.1 (K), D60.1 (K), D61.1 (K), D62.1 (K), D63.1 (K), D64.1 (K), D65.1 (K), D7.1 (K), D8.1 (K), D9.1 (K), J1.S, J10.S, J11.S, J12.S, J13.S, J14.S, J15.S, J16.S, J17.S, J18.S, J19.S, J20.S, J21.S, J22.1, J3.S, J4.S, J5.S, J6.S, J7.S, J8.S, J9.S, R10.2, R11.2, R12.2, R13.2, R14.2, R15.2, R16.2, R17.2, R18.2, R19.2, R20.2, R21.2, R22.2, R23.2, R24.2, R25.2, R3.2, R5.2, R6.2, R8.2, R9.2, U1.18 (AD0), U1.24 (AD1), U1.25 (GND), U1.9 (GND), U10.18 (AD0), U10.25 (GND), U10.9 (GND), U11.25 (GND), U11.9 (GND), U2.24 (AD1), U2.25 (GND), U2.9 (GND), U3.5 (GND), U6.10 (DS), U6.15 (~{CE}), U6.8 (GND), U7.15 (~{CE}), U7.8 (GND), U8.15 (~{CE}), U8.8 (GND), U9.15 (~{CE}), U9.8 (GND)
- new net EG_MODESELECT: R14.1, SW4.1, U8.11 (D0)
- new net EG_OUTPUT_PATCH: A1.25 (ADC_3), D12.2 (A)
- new net EG_TRIGGERSELECT: R13.1, SW3.1, U9.6 (D7)
- new net LPG_GATE1MODE: R22.1, SW12.1, U7.11 (D0)
- new net LPG_GATE2MODE: R23.1, SW13.1, U7.12 (D1)
- new net LPG_LEVEL1CTRL: D28.1 (K), U6.4 (D5)
- new net LPG_LEVEL2CTRL: D29.1 (K), U6.5 (D6)
- new net MASTER: C30.1, RV28.2, U5.20 (I11)
- new net MODOSC_FREQCTRL: D24.1 (K), U6.12 (D1)
- new net MODOSC_MODCTROL: D25.1 (K), U6.13 (D2)
- new net MODOSC_MODULATIONMODE: R17.1, SW7.1, U8.14 (D3)
- new net MODOSC_WAVEFORMTOGGLE: R18.1, SW8.1, U8.3 (D4)
- new net OSCILLATOR_MIDITOGGLE: R21.1, SW9.1, U8.6 (D7)
- new net PL: A1.8 (SPI1_CS), U6.1 (~{PL}), U7.1 (~{PL}), U8.1 (~{PL}), U9.1 (~{PL})
- new net PLSR_MODE: R16.1, SW6.1, U8.13 (D2)
- new net PLSR_PERIODCTRL: D23.1 (K), U6.11 (D0)
- new net PLSR_TRIGGERSELECT: R15.1, SW5.1, U8.12 (D1)
- new net RNDMVOLTAGE_TRIG: R24.1, SW14.1, U7.13 (D2)
- new net SDA: A1.13 (I2C1_SDA), R27.2, U1.20 (SDA), U10.20 (SDA), U11.20 (SDA), U2.20 (SDA)
- new net SEQ_STAGES: R6.1, SW2.1, U9.12 (D1)
- new net SEQ_TRIGGERSELECT: R5.1, SW1.1, U9.11 (D0)
- new net SQ_TOGGLESTEP1: R8.1, SW16.2 (B), U9.13 (D2)
- new net SQ_TOGGLESTEP2: R9.1, SW17.2 (B), U9.14 (D3)
- new net SQ_TOGGLESTEP3: R10.1, SW18.2 (B), U9.3 (D4)
- new net SQ_TOGGLESTEP4: R11.1, SW19.2 (B), U9.4 (D5)
- new net SQ_TOGGLESTEP5: R12.1, SW20.2 (B), U9.5 (D6)
- no-connect marks 13 -> 24
Other:
- note added: "+VE"
- note added: "-VE"
- note added: "0x58"
- note added: "0x59"
- note added: "0x5A"
- note added: "0x5B"
- note added: "3"
- note added: "4"
- note added: "5"
- note added: "AM"
- note added: "BUTTON CONTROL"
- note added: "CLOCK"
- note added: "CLOCK SYNC MODE"
- note added: "CLOCK TRIGGER INDICATOR"
- note added: "COMBI"
- note added: "COMPLEX OSC POLARITY"
- note added: "COMPLEX OSC WAVEFORM"
- note added: "EG MODE"
- note added: "EG TRIGGER INDICATOR"
- note added: "EG TRIGGER MODES"
- note added: "FM"
- note added: "FREE"
- note added: "LED DRIVERS"
- note added: "LO PASS"
- note added: "LPG 1 MODES"
- note added: "LPG 1 TRIGGER INDICATOR"
- note added: "LPG 2 MODES"
- note added: "MIDI"
- note added: "MIDI OFF"
- note added: "MIDI ON"
- note added: "MOD OSC MODULATION MODE"
- note added: "MOD OSC WAVEFORM"
- note added: "MUX"
- note added: "OSCILLATING"
- note added: "OSCILLATOR MIDI TOGGLE"
- note added: "PATCH BAY"
- note added: "POTS"
- note added: "PULSAR"
- note added: "PULSAR SYNC MODES"
- note added: "PULSAR TRIGGER INDICATOR"
- note added: "PULSAR TRIGGER MODES"
- note added: "RNDM VOLTAGE TRIGGER INDICATOR"
- note added: "RNDM VOLTAGE TRIGGER MODE"
- note added: "SAWTOOTH"
- note added: "SEQ"
- note added: "SEQ STAGES"
- note added: "SEQ STEPS"
- note added: "SEQ TRIGGER MODES"
- note added: "SEQUENCER"
- note added: "SHIFT REGISTERS"
- note added: "SINE"
- note added: "SQUARE"
- note added: "STEP 1"
- note added: "STEP 2"
- note added: "STEP 3"
- note added: "STEP 4"
- note added: "STEP 5"
- note added: "SUSTAIN"
- note added: "SYNC"
- note added: "TRANSIENT"
- note added: "TRI"
- note added: "VCA"
- note removed: "BUTTON CONTROL MATRIX"
- note removed: "MUX_1"
- note removed: "MUX_2"
- note removed: "VIRTUAL MODULAR MATRIX"
- moved on the sheet: A1, D1, D23, D24, D25, D26, D27, D28, D29, J1, J15, J16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

Commit message: PCB Footprint Updates
- changed 6N138 to DIP-8 package
Parts:
- D2: footprint PCM_Diode_SMD_AKL:D_1206_3216Metric_Pad1.42x1.75mm_HandSolder -> Diode_SMD:D_SOD-123
- U3: footprint Package_SO:SOP-8_6.62x9.15mm_P2.54mm -> Package_DIP:DIP-8_W7.62mm_LongPads
Changed lines of the file:
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@@
 			)
 		)
-		(property "Footprint" "Package_SO:SOP-8_6.62x9.15mm_P2.54mm"
+		(property "Footprint" "Package_DIP:DIP-8_W7.62mm_LongPads"
 			(at 314.706 54.61 0)
 			(effects
@@
 			)
 		)
-		(property "Footprint" "PCM_Diode_SMD_AKL:D_1206_3216Metric_Pad1.42x1.75mm_HandSolder"
+		(property "Footprint" "Diode_SMD:D_SOD-123"
 			(at 68.58 46.99 0)
 			(effects
