File: build/WEASEL_KiCad/WEASEL_KiCad_MainBoard.kicad_pcb (KiCad board)
At the start: 2 copper layers, 335 x 200 mm, 224 parts, among them J1 MIDI IN, J10 PLSR_OUTPUT2, J11 PLSR_OUTPUT3, J12 RNDM_OUTPUT1, J13 RNDM_OUTPUT2, J14 RNDM_OUTPUT3, J15 PLSR_PERIODCTRL, J16 MODOSC_FREQCTRL, J17 MODOSC_MODCTRL, J18 COMPOSC_PITCHCTRL, J19 COMPOSC_WAVEFOLDERCTRL, J2 STEREO_OUTPUT, J20 LPG_LEVEL1CTRL, J21 LPG_LEVEL2CTRL, J22 Jack-DC, J3 SEQ_OUTPUT1, J4 SEQ_OUTPUT2, J5 SEQ_OUTPUT3, J6 EG_OUTPUT1, J7 EG_OUTPUT2, J8 EG_OUTPUT3, J9 PLSR_OUTPUT1, SW1 SEQ_TRIGGERSELECT, SW10 COMPLEXOSC_POLARITY, SW11 COMPLEXOSC_WAVETOGGLE, SW12 LPG_GATE1MODE, SW13 LPG_GATE2MODE, SW14 RNDMVOLTAGE_TRIGGERSELECT, SW15 CLOCK_SYNCTOGGLE, SW16 SQ_TOGGLESTEP1, SW17 SQ_TOGGLESTEP2, SW18 SQ_TOGGLESTEP3, SW19 SQ_TOGGLESTEP4, SW2 SEQ_STAGES, SW20 SQ_TOGGLESTEP5, SW3 EG_TRIGGERSELECT, SW4 EG_MODESELECT, SW5 PLSR_TRIGGERSELECT, SW6 PLSR_MODE, SW7 MODOSC_MODULATIONMODE, SW8 MODOSC_WAVEFORMTOGGLE, SW9 OSCILLATOR_MIDITOGGLE, U1 AW9523B, U10 AW9523B, U11 AW9523B, U2 AW9523B, U3 6N138, U4 CD74HC4067M, U5 CD74HC4067M, U6 74HC165, U7 74HC165, U8 74HC165, U9 74HC165

Commit message: PCB Footprint Updates
- changed 6N138 to DIP-8 package
Parts:
- removed the REF** at (255.5, 29.3)
- removed the REF** at (30.5, 29.3)
- removed the REF** at (130.5, 29.3)
- removed the REF** at (130.5, 219.3)
- removed the REF** at (30.5, 219.3)
- removed the REF** at (355.5, 29.3)
- removed the REF** at (355.5, 219.3)
- removed the REF** at (255.5, 219.3)
- added REF**: MountingHole_2.2mm_M2, MountingHole:MountingHole_2.2mm_M2, F.Cu at (365.1, 228.5)
- added REF**: MountingHole_2.2mm_M2, MountingHole:MountingHole_2.2mm_M2, F.Cu at (140.1, 228.5)
- added REF**: MountingHole_2.2mm_M2, MountingHole:MountingHole_2.2mm_M2, F.Cu at (265.1, 38.5)
- added REF**: MountingHole_2.2mm_M2, MountingHole:MountingHole_2.2mm_M2, F.Cu at (40.1, 228.5)
- added REF**: MountingHole_2.2mm_M2, MountingHole:MountingHole_2.2mm_M2, F.Cu at (265.1, 228.5)
- added REF**: MountingHole_2.2mm_M2, MountingHole:MountingHole_2.2mm_M2, F.Cu at (40.1, 38.5)
- added REF**: MountingHole_2.2mm_M2, MountingHole:MountingHole_2.2mm_M2, F.Cu at (140.1, 38.5)
- added REF**: MountingHole_2.2mm_M2, MountingHole:MountingHole_2.2mm_M2, F.Cu at (365.1, 38.5)
- D2: footprint PCM_Diode_SMD_AKL:D_1206_3216Metric_Pad1.42x1.75mm_HandSolder -> Diode_SMD:D_SOD-123
- U3: footprint Package_SO:SOP-8_6.62x9.15mm_P2.54mm -> Package_DIP:DIP-8_W7.62mm_LongPads
- moved U3 14.0 mm to (136.0, 53.4)
- moved C41 13.3 mm to (318.6, 147.2)
- moved D53 13.3 mm to (301.3, 149.3)
- moved D59 13.3 mm to (306.6, 162.9)
- moved D61 13.3 mm to (306.6, 166.3)
- moved J11 13.3 mm to (285.1, 201.3)
- moved J14 13.3 mm to (285.1, 215.8)
- moved J20 13.3 mm to (257.6, 207.8)
- moved J21 13.3 mm to (270.1, 207.8)
- moved C11 13.3 mm to (271.9, 114.5)
- moved C12 13.3 mm to (293.6, 111.2)
- moved C24 13.3 mm to (300.4, 110.8)
- moved C25 13.3 mm to (316.8, 114.5)
- moved C26 13.3 mm to (329.3, 114.5)
- moved C27 13.3 mm to (341.8, 114.5)
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Routing:
- net MIDI_INPUT: track 186.0 -> 204.8 mm
- net Net-(U3-VO1): track 10.6 -> 6.70 mm
- net DGND: track 346.2 -> 347.8 mm

Commit message: PCB Revisions
Parts:
- removed the REF** at (365.1, 228.5)
- removed the REF** at (140.1, 228.5)
- removed the REF** at (265.1, 38.5)
- removed the REF** at (40.1, 228.5)
- removed the REF** at (265.1, 228.5)
- removed the REF** at (40.1, 38.5)
- removed the REF** at (140.1, 38.5)
- removed the REF** at (365.1, 38.5)
- added REF**: MountingHole_2.2mm_M2, MountingHole:MountingHole_2.2mm_M2, F.Cu at (269.1, 226.8)
- added REF**: MountingHole_2.2mm_M2, MountingHole:MountingHole_2.2mm_M2, F.Cu at (369.1, 226.8)
- added REF**: MountingHole_2.2mm_M2, MountingHole:MountingHole_2.2mm_M2, F.Cu at (44.1, 226.8)
- added REF**: MountingHole_2.2mm_M2, MountingHole:MountingHole_2.2mm_M2, F.Cu at (369.1, 36.8)
- added REF**: MountingHole_2.2mm_M2, MountingHole:MountingHole_2.2mm_M2, F.Cu at (144.1, 226.8)
- added REF**: MountingHole_2.2mm_M2, MountingHole:MountingHole_2.2mm_M2, F.Cu at (44.1, 36.8)
- added REF**: MountingHole_2.2mm_M2, MountingHole:MountingHole_2.2mm_M2, F.Cu at (144.1, 36.8)
- added REF**: MountingHole_2.2mm_M2, MountingHole:MountingHole_2.2mm_M2, F.Cu at (269.1, 36.8)
- moved D32 4.39 mm to (271.9, 47.1)
- moved D33 4.39 mm to (271.9, 48.9)
- moved D34 4.39 mm to (271.9, 50.5)
- moved D35 4.39 mm to (271.9, 64.3)
- moved D36 4.39 mm to (271.9, 67.5)
- moved D37 4.39 mm to (290.9, 56.8)
- moved D54 4.39 mm to (294.2, 172.8)
- moved D55 4.39 mm to (295.9, 172.8)
- moved D64 4.39 mm to (313.9, 130.3)
- moved D65 4.39 mm to (328.4, 137.1)
- moved D63 4.39 mm to (313.9, 127.0)
- moved D50 4.39 mm to (172.6, 126.5)
- moved C1 4.39 mm to (109.6, 126.0)
- moved C10 4.39 mm to (255.9, 112.8)
- moved C13 4.39 mm to (157.1, 173.8)
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