File: build/WEASEL_KiCad/WEASEL_KiCad_PANELS.kicad_pcb (KiCad board)
At the start: 2 copper layers, 335 x 400 mm, 90 parts

Commit message: PCB Revisions
Parts:
- removed the ? at (292.1, 97.2)
- removed the ? at (292.2, 114.7)
- removed the G*** at (97.3, 98.2) (x2)
- removed the G*** at (97.3, 98.1)
- removed the G*** at (207.5, 380.6) (x2)
- removed the REF** at (247.9, 269.5)
- removed the REF** at (125.4, 255.0)
- removed the REF** at (297.1, 211.7)
- removed the REF** at (270.1, 223.8)
- removed the REF** at (189.6, 114.5)
- removed the REF** at (45.4, 275.7)
- removed the REF** at (297.1, 176.7)
- removed the REF** at (317.4, 105.7)
- removed the REF** at (270.4, 85.7)
- removed the REF** at (207.9, 261.5)
- removed the REF** at (214.6, 97.1)
- removed the REF** at (200.1, 223.8)
- removed the REF** at (145.4, 85.7)
- removed the REF** at (212.6, 158.8)
- removed the REF** at (257.6, 223.8)
- removed the REF** at (167.1, 176.7)
- removed the REF** at (177.1, 114.5)
- removed the REF** at (232.6, 223.8)
- removed the REF** at (167.9, 255.0)
- removed the REF** at (349.7, 176.7)
- removed the REF** at (140.4, 262.0)
- removed the REF** at (290.1, 158.8)
- removed the REF** at (275.4, 261.5)
- removed the REF** at (187.6, 158.8)
- removed the REF** at (277.6, 158.8)
- removed the REF** at (45.4, 285.7)
- removed the REF** at (290.4, 269.5)
- removed the REF** at (175.1, 223.8)
- removed the REF** at (349.6, 238.7)
- removed the REF** at (184.6, 176.7)
- removed the REF** at (187.6, 223.8)
- removed the REF** at (245.1, 158.8)
- removed the REF** at (145.4, 475.7)
- removed the REF** at (262.9, 261.5)
- removed the REF** at (235.4, 269.8)
- removed the REF** at (270.4, 285.7)
- removed the REF** at (145.4, 285.7)
- removed the REF** at (335.1, 158.8)
- removed the REF** at (220.4, 261.5)
- removed the REF** at (202.1, 176.7)
- removed the REF** at (200.1, 158.8)
- removed the REF** at (202.4, 114.8)
- removed the REF** at (270.4, 275.7)
- removed the REF** at (164.6, 114.5)
- removed the REF** at (145.4, 275.7)
- removed the REF** at (189.6, 97.0)
- removed the REF** at (155.4, 269.5)
- removed the REF** at (245.1, 223.8)
- removed the REF** at (162.6, 158.8)
- removed the REF** at (341.6, 105.7)
- removed the REF** at (270.4, 475.7)
- removed the REF** at (125.4, 269.5)
- removed the REF** at (370.4, 275.7)
- removed the REF** at (232.6, 158.8)
- removed the REF** at (370.4, 475.7)
- removed the REF** at (347.6, 158.8)
- removed the REF** at (370.4, 85.7)
- removed the REF** at (45.4, 475.7)
- removed the REF** at (45.4, 85.7)
- removed the REF** at (162.6, 223.8)
- removed the REF** at (259.6, 97.1)
- removed the REF** at (297.1, 194.2)
- removed the REF** at (370.4, 285.7)
- removed the REF** at (247.9, 255.0)
- removed the REF** at (257.6, 158.8)
- removed the REF** at (322.6, 158.8)
- removed the REF** at (290.4, 255.0)
- removed the REF** at (235.4, 255.2)
- removed the REF** at (167.9, 269.5)
- removed the REF** at (155.4, 255.0)
- removed the REF** at (175.1, 158.8)
- removed the REF** at (195.4, 261.5)
- removed the REF** at (182.9, 261.5)
- removed the REF** at (234.7, 176.6)
- removed the REF** at (214.6, 114.8)
- removed the REF** at (259.7, 114.6)
- removed the REF** at (329.6, 211.7)
- removed the REF** at (272.1, 176.6)
- removed the REF** at (310.1, 158.8)
- removed the REF** at (329.6, 176.7)
- added ?: , , F.Cu at (281.4, 91.8)
- added ?: , , F.Cu at (281.3, 74.3)
- added G*** (x3): LOGO, AXS_LOGO_KICAD:AXS_LOGO_FMASK_10X10, F.Cu at (86.5, 75.3)
- added G*** (x2): LOGO, WEASEL:WEASEL_FMASK_fullsize, F.Cu at (196.7, 357.8)
- added REF**: button, SimpleSynthPanel:Panel Jack, F.Cu at (173.8, 153.8)
- added REF**: Panel Jack, SimpleSynthPanel:Panel Jack, F.Cu at (224.6, 246.9)
- added REF**: Panel Jack, SimpleSynthPanel:Panel Jack, F.Cu at (279.6, 246.6)
- added REF**: Panel Fader Slide Pot, SimpleSynthPanel:Panel Fader Slide Pot, F.Cu at (324.3, 135.9)
- added REF**: Panel Fader Slide Pot, SimpleSynthPanel:Panel Fader Slide Pot, F.Cu at (246.8, 200.9)
- added REF**: MountingHole_2.2mm_M2, MountingHole:MountingHole_2.2mm_M2, F.Cu at (134.6, 452.9)
- added REF**: button, SimpleSynthPanel:Panel Jack, F.Cu at (178.8, 74.1)
- added REF**: Panel Jack, SimpleSynthPanel:Panel Jack, F.Cu at (252.1, 238.6)
- added REF**: Panel Jack, SimpleSynthPanel:Panel Jack, F.Cu at (129.6, 239.1)
- added REF**: Panel Fader Slide Pot, SimpleSynthPanel:Panel Fader Slide Pot, F.Cu at (234.3, 135.9)
- added REF**: button, SimpleSynthPanel:Panel Jack, F.Cu at (286.3, 153.8)
- added REF**: SPDT, SimpleSynthPanel:Panel Jack, F.Cu at (203.8, 91.9)
- added REF**: Panel Jack, SimpleSynthPanel:Panel Jack, F.Cu at (197.1, 238.6)
- added REF**: Panel Jack, SimpleSynthPanel:Panel Jack, F.Cu at (279.6, 232.1)
- added REF**: MountingHole_2.2mm_M2, MountingHole:MountingHole_2.2mm_M2, F.Cu at (34.6, 252.9)
- added REF**: Panel Jack, SimpleSynthPanel:Panel Jack, F.Cu at (264.6, 238.6)
- added REF**: MountingHole_2.2mm_M2, MountingHole:MountingHole_2.2mm_M2, F.Cu at (259.6, 62.9)
- added REF**: button, SimpleSynthPanel:Panel Jack, F.Cu at (318.8, 153.9)
- added REF**: Panel Jack, SimpleSynthPanel:Panel Jack, F.Cu at (114.6, 232.1)
- added REF**: Panel Fader Slide Pot, SimpleSynthPanel:Panel Fader Slide Pot, F.Cu at (189.3, 135.9)
- added REF**: Panel Fader Slide Pot, SimpleSynthPanel:Panel Fader Slide Pot, F.Cu at (266.8, 135.9)
- added REF**: Panel Jack, SimpleSynthPanel:Panel Jack, F.Cu at (157.1, 246.6)
- added REF**: MountingHole_2.2mm_M2, MountingHole:MountingHole_2.2mm_M2, F.Cu at (359.6, 262.9)
- added REF**: Panel Knob 1P, SimpleSynthPanel:Panel Knob 1P, F.Cu at (338.9, 153.9)
- added REF**: SPDT, SimpleSynthPanel:Panel Jack, F.Cu at (153.8, 91.6)
- added REF**: Panel Fader Slide Pot, SimpleSynthPanel:Panel Fader Slide Pot, F.Cu at (311.8, 135.9)
- added REF**: Panel Fader Slide Pot, SimpleSynthPanel:Panel Fader Slide Pot, F.Cu at (164.3, 200.9)
- added REF**: Panel Fader Slide Pot, SimpleSynthPanel:Panel Fader Slide Pot, F.Cu at (176.8, 200.9)
- added REF**: SPDT, SimpleSynthPanel:Panel Jack, F.Cu at (166.3, 91.6)
- added REF**: button, SimpleSynthPanel:Panel Jack, F.Cu at (203.8, 74.3)
- added REF**: Panel Fader Slide Pot, SimpleSynthPanel:Panel Fader Slide Pot, F.Cu at (246.8, 135.9)
- added REF**: Panel Knob 1P, SimpleSynthPanel:Panel Knob 1P, F.Cu at (338.8, 215.9)
- added REF**: MountingHole_2.2mm_M2, MountingHole:MountingHole_2.2mm_M2, F.Cu at (259.6, 452.9)
- added REF**: button, SimpleSynthPanel:Panel Jack, F.Cu at (286.3, 188.8)
- added REF**: Panel Jack, SimpleSynthPanel:Panel Jack, F.Cu at (237.1, 246.6)
- added REF**: SPDT, SimpleSynthPanel:Panel Jack, F.Cu at (178.8, 91.6)
- added REF**: Panel Jack, SimpleSynthPanel:Panel Jack, F.Cu at (224.6, 232.4)
- added REF**: MountingHole_2.2mm_M2, MountingHole:MountingHole_2.2mm_M2, F.Cu at (259.6, 252.9)
- added REF**: button, SimpleSynthPanel:Panel Jack, F.Cu at (156.3, 153.8)
- added REF**: Panel Jack, SimpleSynthPanel:Panel Jack, F.Cu at (184.6, 238.6)
- added REF**: Panel Jack, SimpleSynthPanel:Panel Jack, F.Cu at (172.1, 238.6)
- added REF**: button, SimpleSynthPanel:Panel Jack, F.Cu at (248.9, 91.8)
- added REF**: MountingHole_2.2mm_M2, MountingHole:MountingHole_2.2mm_M2, F.Cu at (359.6, 252.9)
- added REF**: Panel Fader Slide Pot, SimpleSynthPanel:Panel Fader Slide Pot, F.Cu at (259.3, 200.9)
- added REF**: Panel Jack, SimpleSynthPanel:Panel Jack, F.Cu at (144.6, 232.1)
- added REF**: MountingHole_2.2mm_M2, MountingHole:MountingHole_2.2mm_M2, F.Cu at (34.6, 62.9)
- added REF**: MountingHole_2.2mm_M2, MountingHole:MountingHole_2.2mm_M2, F.Cu at (359.6, 452.9)
- added REF**: MountingHole_2.2mm_M2, MountingHole:MountingHole_2.2mm_M2, F.Cu at (134.6, 62.9)
- added REF**: Panel Knob 1P, SimpleSynthPanel:Panel Knob 1P, F.Cu at (223.9, 153.8)
- added REF**: button, SimpleSynthPanel:Panel Jack, F.Cu at (330.8, 82.9)
- added REF**: SPDT, SimpleSynthPanel:Panel Jack, F.Cu at (191.6, 91.9)
- added REF**: Panel Fader Slide Pot, SimpleSynthPanel:Panel Fader Slide Pot, F.Cu at (164.3, 135.9)
- added REF**: Panel Jack, SimpleSynthPanel:Panel Jack, F.Cu at (144.6, 246.6)
- added REF**: Panel Fader Slide Pot, SimpleSynthPanel:Panel Fader Slide Pot, F.Cu at (151.8, 135.9)
- added REF**: Panel Fader Slide Pot, SimpleSynthPanel:Panel Fader Slide Pot, F.Cu at (189.3, 200.9)
- added REF**: MountingHole_2.2mm_M2, MountingHole:MountingHole_2.2mm_M2, F.Cu at (34.6, 452.9)
- added REF**: button, SimpleSynthPanel:Panel Jack, F.Cu at (286.3, 171.3)
- added REF**: Panel Fader Slide Pot, SimpleSynthPanel:Panel Fader Slide Pot, F.Cu at (279.3, 135.9)
- added REF**: button, SimpleSynthPanel:Panel Jack, F.Cu at (318.8, 188.8)
- added REF**: Panel Fader Slide Pot, SimpleSynthPanel:Panel Fader Slide Pot, F.Cu at (151.8, 200.9)
- added REF**: MountingHole_2.2mm_M2, MountingHole:MountingHole_2.2mm_M2, F.Cu at (134.6, 262.9)
- added REF**: Panel Knob 1P, SimpleSynthPanel:Panel Knob 1P, F.Cu at (191.3, 153.9)
- added REF**: button, SimpleSynthPanel:Panel Jack, F.Cu at (306.6, 82.9)
- added REF**: MountingHole_2.2mm_M2, MountingHole:MountingHole_2.2mm_M2, F.Cu at (134.6, 252.9)
- added REF**: Panel Jack, SimpleSynthPanel:Panel Jack, F.Cu at (157.1, 232.1)
- added REF**: Panel Fader Slide Pot, SimpleSynthPanel:Panel Fader Slide Pot, F.Cu at (201.8, 135.9)
- added REF**: button, SimpleSynthPanel:Panel Jack, F.Cu at (248.8, 74.3)
- added REF**: MountingHole_2.2mm_M2, MountingHole:MountingHole_2.2mm_M2, F.Cu at (359.6, 62.9)
- added REF**: Panel Jack, SimpleSynthPanel:Panel Jack, F.Cu at (114.6, 246.6)
- added REF**: Panel Fader Slide Pot, SimpleSynthPanel:Panel Fader Slide Pot, F.Cu at (299.3, 135.9)
- added REF**: Panel Jack, SimpleSynthPanel:Panel Jack, F.Cu at (237.1, 232.1)
- added REF**: Panel Jack, SimpleSynthPanel:Panel Jack, F.Cu at (209.6, 238.6)
- added REF**: Panel Fader Slide Pot, SimpleSynthPanel:Panel Fader Slide Pot, F.Cu at (336.8, 135.9)
- added REF**: Panel Fader Slide Pot, SimpleSynthPanel:Panel Fader Slide Pot, F.Cu at (221.8, 135.9)
- added REF**: Panel Fader Slide Pot, SimpleSynthPanel:Panel Fader Slide Pot, F.Cu at (176.8, 135.9)
- added REF**: Panel Fader Slide Pot, SimpleSynthPanel:Panel Fader Slide Pot, F.Cu at (221.8, 200.9)
- added REF**: Panel Knob 1P, SimpleSynthPanel:Panel Knob 1P, F.Cu at (261.3, 153.8)
- added REF**: MountingHole_2.2mm_M2, MountingHole:MountingHole_2.2mm_M2, F.Cu at (34.6, 262.9)
- added REF**: MountingHole_2.2mm_M2, MountingHole:MountingHole_2.2mm_M2, F.Cu at (259.6, 262.9)
- added REF**: Panel Fader Slide Pot, SimpleSynthPanel:Panel Fader Slide Pot, F.Cu at (234.3, 200.9)
- moved G*** 25.3 mm to (196.5, 357.7)
- moved REF** 25.3 mm to (338.9, 183.9)
- moved G*** 25.3 mm to (87.1, 181.9)
Other:
- outline, holes or cut-outs redrawn
